File: Load_Balancer_mk_4.kicad_pcb (KiCad board)
At the start: 2 copper layers, 100 x 70 mm, 44 parts, among them J1 Screw_Terminal_01x01, J2 Screw_Terminal_01x01, J3 Screw_Terminal_01x01, J4 Screw_Terminal_01x01, Q1 2N4403, Q2 2N4403, U1 4011, U2 4013

Commit message: Add some silkscreen text
Other:
- board text added: "(C) ADAM CORDINGLEY 2021"
- board text added: "120VAC MAX!!"
- board text added: "MAINS SOURCE BALANCER"
- board text added: "www.acordingley.us"
